Commit message: Revert "Model Loading and Conversion"

File: models/pendulum/pendulum.urdf (robot description, URDF)
Before this commit: robot pendulum, 2 links, 1 joints
Links:
- link base: mass 2 -> None
Joints:
- added joint fixed_joint: type fixed, parent world, child base, origin xyz=0 0 0 rpy=0 0 0

Commit message: fix pendulum geometries and inertias

File: models/pendulum/pendulum.urdf (robot description, URDF)
Before this commit: robot pendulum, 2 links, 1 joints
Links:
- link base: geometry visual sphere radius=0.03
- link pendulum_link: geometry collision capsule length=1.0 radius=0.02; visual capsule length=1.0 radius=0.02
Joints:
- joint pendulum_joint: axis 0 0 1 -> 0 1 0

Commit message: changed comments to be about merging #21 instead of mistaken mjx bug

File: models/pendulum/pendulum.urdf (robot description, URDF)
Before this commit: robot pendulum, 2 links, 1 joints
Links:
- link base: geometry 
- link pendulum_link: geometry collision cylinder length=1.0 radius=0.02; visual cylinder length=1.0 radius=0.02
Joints:
- joint pendulum_joint: axis 0 1 0 -> 0 0 1
